Commit message: working simulation

File: src/alex/urdf/alex.urdf.xacro (robot description, xacro)
@@ -1,8 +1,13 @@
 <?xml version="1.0" ?>
 <robot name="alex">
-    <link name="base_footprint">
+	<link name="base_footprint">
+		<origin xyz="0 0 0" rpy="0 0 0"/>
     </link>
     <!-- Define the chassis link -->
     <link name="base_link">
+        <inertial>
+            <mass value="7.416800635961257"/>
+            <inertia ixx="0.03775" iyy="0.010039" izz="0.045988" ixy="1e-06" iyz="2.1e-05" ixz="-0.0"/>
+        </inertial>
         <visual>
             <geometry>
@@ -29,49 +34,94 @@
             </material>
         </visual>
+        <collision>
+            <geometry>
+                <box size="0.01 0.100 0.020"/>
+            </geometry>
+        </collision>
     </link>
     <!-- Define the wheel link -->
     <link name="front_left_wheel_link">
-        <visual>
-            <origin rpy="1.57 0 0" xyz="0 0 0" />
-            <geometry>
-                <cylinder length="0.028" radius="0.034"/>
-            </geometry>
-            <material name="black">
-                <color rgba="0.2 0.2 0.2 1.0"/>
-            </material>
-        </visual>
+        <inertial>
+            <mass value="0.09794643947061814"/>
+            <inertia ixx="5.7e-05" iyy="3.5e-05" izz="3.5e-05" ixy="-0.0" iyz="-0.0" ixz="0.0"/>
+        </inertial>
+        <visual>
+            <origin rpy="1.57 0 0" xyz="0 0 0" />
+            <geometry>
+                <cylinder length="0.028" radius="0.034"/>
+            </geometry>
+            <material name="black">
+                <color rgba="0.2 0.2 0.2 1.0"/>
+            </material>
+        </visual>
+        <collision>
+            <origin rpy="1.57 0 0" xyz="0 0 0" />
+            <geometry>
+                <cylinder length="0.028" radius="0.034"/>
+            </geometry>
+        </collision>
     </link>
     <link name="front_right_wheel_link">
-        <visual>
-            <origin rpy="1.57 0 0" xyz="0 0 0" />
-            <geometry>
-                <cylinder length="0.028" radius="0.034"/>
-            </geometry>
-            <material name="black">
-                <color rgba="0.2 0.2 0.2 1.0"/>
-            </material>
-        </visual>
+        <inertial>
+            <mass value="0.0979464394706181"/>
+            <inertia ixx="5.7e-05" iyy="3.5e-05" izz="3.5e-05" ixy="0.0" iyz="0.0" ixz="0.0"/>
+        </inertial>
+        <visual>
+            <origin rpy="1.57 0 0" xyz="0 0 0" />
+            <geometry>
+                <cylinder length="0.028" radius="0.034"/>
+            </geometry>
+            <material name="black">
+                <color rgba="0.2 0.2 0.2 1.0"/>
+            </material>
+        </visual>
+        <collision>
+            <origin rpy="1.57 0 0" xyz="0 0 0" />
+            <geometry>
+                <cylinder length="0.028" radius="0.034"/>
+            </geometry>
+        </collision>
     </link>
     <link name="rear_left_wheel_link">
-        <visual>
-        <origin rpy="1.57 0 0" xyz="0 0 0" />
-            <geometry>
-                <cylinder length="0.028" radius="0.034"/>
-            </geometry>
-            <material name="black">
-                <color rgba="0.2 0.2 0.2 1.0"/>
-            </material>
-        </visual>
+        <inertial>
+            <mass value="0.0979464394706181"/>
+            <inertia ixx="5.7e-05" iyy="3.5e-05" izz="3.5e-05" ixy="0.0" iyz="0.0" ixz="0.0"/>
+        </inertial>
+        <visual>
+            <origin rpy="1.57 0 0" xyz="0 0 0" />
+            <geometry>
+                <cylinder length="0.028" radius="0.034"/>
+            </geometry>
+            <material name="black">
+                <color rgba="0.2 0.2 0.2 1.0"/>
+            </material>
+        </visual>
+        <collision>
+            <origin rpy="1.57 0 0" xyz="0 0 0" />
+            <geometry>
+                <cylinder length="0.028" radius="0.034"/>
+            </geometry>
+        </collision>
     </link>
     <link name="rear_right_wheel_link">
-        <visual>
-        <origin rpy="1.57 0 0" xyz="0 0 0" />
-            <geometry>
-                <cylinder length="0.028" radius="0.034"/>
-            </geometry>
-            <material name="black">
-                <color rgba="0.2 0.2 0.2 1.0"/>
-            </material>
-        </visual>
+        <inertial>
+            <mass value="0.0979464394706181"/>
+            <inertia ixx="5.7e-05" iyy="3.5e-05" izz="3.5e-05" ixy="0.0" iyz="0.0" ixz="0.0"/>
+        </inertial>
+        <visual>
+            <origin rpy="1.57 0 0" xyz="0 0 0" />
+            <geometry>
+                <cylinder length="0.028" radius="0.034"/>
+            </geometry>
+            <material name="black">
+                <color rgba="0.2 0.2 0.2 1.0"/>
+            </material>
+        </visual>
+        <collision>
+            <origin rpy="1.57 0 0" xyz="0 0 0" />
+            <geometry>
+                <cylinder length="0.028" radius="0.034"/>
+            </geometry>
+        </collision>
     </link>
     <!-- Define link for lidar column-->
@@ -126,4 +176,6 @@
         <origin xyz="-0.058 0.064 0" rpy="0 0 0"/>
         <axis xyz="0 1 0"/>
+        <limit effort="100" velocity="100"/>
+        <dynamics damping="0.0" friction="0.0"/>
     </joint>
     <joint name="rear_right_wheel_joint" type="continuous">
@@ -132,4 +184,6 @@
         <origin xyz="-0.058 -0.064 0" rpy="0 0 0"/>
         <axis xyz="0 1 0"/>
+        <limit effort="100" velocity="100"/>
+        <dynamics damping="0.0" friction="0.0"/>
     </joint>
     <joint name="front_left_wheel_joint" type="continuous">
@@ -138,4 +192,6 @@
         <origin xyz="0.058 0.064 0" rpy="0 0 0"/>
         <axis xyz="0 1 0"/>
+        <limit effort="100" velocity="100"/>
+        <dynamics damping="0.0" friction="0.0"/>
     </joint>
     <joint name="front_right_wheel_joint" type="continuous">
@@ -144,4 +200,53 @@
         <origin xyz="0.058 -0.064 0" rpy="0 0 0"/>
         <axis xyz="0 1 0"/>
-    </joint>
+        <limit effort="100" velocity="100"/>
+        <dynamics damping="0.0" friction="0.0"/>
+    </joint>
+    <!-- Wheel Transmissions -->
+    <transmission name="front_left_wheel_trans">
+        <type>transmission_interface/SimpleTransmission</type>
+        <actuator name="front_left_wheel_motor">
+            <hardwareInterface>EffortJointInterface</hardwareInterface>
+            <mechanicalReduction>1</mechanicalReduction>
+        </actuator>
+        <joint name="front_left_wheel_joint">
+            <hardwareInterface>VelocityJointInterface</hardwareInterface>
+        </joint>
+    </transmission>
+    <transmission name="front_right_wheel_trans">
+        <type>transmission_interface/SimpleTransmission</type>
+        <actuator name="front_right_wheel_motor">
+            <hardwareInterface>EffortJointInterface</hardwareInterface>
+            <mechanicalReduction>1</mechanicalReduction>
+        </actuator>
+        <joint name="front_right_wheel_joint">
+            <hardwareInterface>VelocityJointInterface</hardwareInterface>
+        </joint>
+    </transmission>
+    <transmission name="rear_left_wheel_trans">
+        <type>transmission_interface/SimpleTransmission</type>
+        <actuator name="rear_left_wheel_motor">
+            <hardwareInterface>EffortJointInterface</hardwareInterface>
+            <mechanicalReduction>1</mechanicalReduction>
+        </actuator>
+        <joint name="rear_left_wheel_joint">
+            <hardwareInterface>VelocityJointInterface</hardwareInterface>
+        </joint>
+    </transmission>
+    <transmission name="rear_right_wheel_trans">
+        <type>transmission_interface/SimpleTransmission</type>
+        <actuator name="rear_right_wheel_motor">
+            <hardwareInterface>EffortJointInterface</hardwareInterface>
+            <mechanicalReduction>1</mechanicalReduction>
+        </actuator>
+        <joint name="rear_right_wheel_joint">
+            <hardwareInterface>VelocityJointInterface</hardwareInterface>
+        </joint>
+    </transmission>
+    <!-- ros_control plugin -->
+    <gazebo>
+        <plugin name="gazebo_ros_control" filename="libgazebo_ros_control.so">
+        <robotNamespace>/</robotNamespace>
+        </plugin>
+    </gazebo>
 </robot>
