Commit message: launch files

File: src/alex/urdf/alex.urdf (robot description, URDF)
Before this commit: robot alex, 9 links, 8 joints
Links:
- removed link base_footprint
Joints:
- joint base_joint: parent base_footprint -> (none)

Commit message: fixed robot description

File: src/alex/urdf/alex.urdf (robot description, URDF)
Before this commit: robot alex, 8 links, 8 joints
Links:
- added link world
Joints:
- joint base_joint: parent (none) -> world

Commit message: map directory and urdf update for clearance

File: src/alex/urdf/alex.urdf (robot description, URDF)
Before this commit: robot alex, 9 links, 8 joints
Links:
- added link color_sensor_link; visual box size=0.045 0.045 0.045
- added link rear_link; visual box size=0.06 0.100 0.020
Joints:
- added joint color_sensor_joint: type fixed, parent front_link, child color_sensor_link, origin xyz=0.015 0 0 rpy=0 0 0
- added joint rear_joint: type fixed, parent base_link, child rear_link, origin xyz=-0.155 0 0 rpy=0 0 0
